File: STM32_FlightController_Rev2/STM32_FlightController.kicad_pcb (KiCad board)
At the start: 4 copper layers, 42 x 44.4 mm, 56 parts, among them J1 629105150521, J2 JST_SH_SM08B-SRSS-TB_1x08-1MP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, J3 JST_SH_SM04B-SRSS-TB_1x04-1MP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, J4 JST_SH_SM04B-SRSS-TB_1x04-1MP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, J5 Conn_02x05_Odd_Even, SW1 PTS815SJM250SMTRLFS, SW2 PCM12SMTR, U1 SN74LVC1T45DBV, U2 ICM-20948, U3 STM32F405RGTx, U4 USBLC6-2SC6, U5 AMS1117-3.3, U6 TLV70018, U7 BMP390L, U8 SN74LVC1T45DBV, Y1 X32258MOB4SI

Commit message: correct PCB traces regarding TIM pins
Connections:
- U3 pad 20: /S4 -> unconnected-(U3-PA4-Pad20)
- U3 pad 21: /S3 -> unconnected-(U3-PA5-Pad21)
- U3 pad 22: /S2 -> /S4
- U3 pad 23: /S1 -> /S3
- U3 pad 26: unconnected-(U3-PB0-Pad26) -> /S2
- U3 pad 27: unconnected-(U3-PB1-Pad27) -> /S1
Changed lines of the file:
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@@
 	(net 75 "unconnected-(U3-PC15-Pad4)")
 	(net 76 "unconnected-(U3-PA0-Pad14)")
-	(net 77 "unconnected-(U3-PB0-Pad26)")
+	(net 77 "unconnected-(U3-PA4-Pad20)")
 	(net 78 "unconnected-(U3-PC4-Pad24)")
 	(net 79 "unconnected-(U3-PA10-Pad43)")
-	(net 80 "unconnected-(U3-PB1-Pad27)")
+	(net 80 "unconnected-(U3-PA5-Pad21)")
 	(net 81 "unconnected-(U3-PC2-Pad10)")
 	(net 82 "unconnected-(U3-PC5-Pad25)")
@@
 			(layers "F.Cu" "F.Mask" "F.Paste")
 			(roundrect_rratio 0.25)
-			(net 39 "/S4")
+			(net 77 "unconnected-(U3-PA4-Pad20)")
 			(pinfunction "PA4")
-			(pintype "bidirectional")
+			(pintype "bidirectional+no_connect")
 		)
 		(pad "21" smd roundrect
@@
 			(layers "F.Cu" "F.Mask" "F.Paste")
 			(roundrect_rratio 0.25)
-			(net 38 "/S3")
+			(net 80 "unconnected-(U3-PA5-Pad21)")
 			(pinfunction "PA5")
-			(pintype "bidirectional")
+			(pintype "bidirectional+no_connect")
 		)
 		(pad "22" smd roundrect
@@
 			(layers "F.Cu" "F.Mask" "F.Paste")
 			(roundrect_rratio 0.25)
-			(net 37 "/S2")
+			(net 39 "/S4")
 			(pinfunction "PA6")
 			(pintype "bidirectional")
@@
 			(layers "F.Cu" "F.Mask" "F.Paste")
 			(roundrect_rratio 0.25)
-			(net 36 "/S1")
+			(net 38 "/S3")
 			(pinfunction "PA7")
 			(pintype "bidirectional")
@@
 			(layers "F.Cu" "F.Mask" "F.Paste")
 			(roundrect_rratio 0.25)
-			(net 77 "unconnected-(U3-PB0-Pad26)")
+			(net 37 "/S2")
 			(pinfunction "PB0")
-			(pintype "bidirectional+no_connect")
+			(pintype "bidirectional")
 		)
 		(pad "27" smd roundrect
@@
 			(layers "F.Cu" "F.Mask" "F.Paste")
 			(roundrect_rratio 0.25)
-			(net 80 "unconnected-(U3-PB1-Pad27)")
+			(net 36 "/S1")
 			(pinfunction "PB1")
-			(pintype "bidirectional+no_connect")
+			(pintype "bidirectional")
 		)
 		(pad "28" smd roundrect
@@
 	)
 	(segment
-		(start 35.2625 44.1625)
-		(end 35.2625 43.1375)
+		(start 37.2625 46.7375)
+		(end 35.5125 48.4875)
 		(width 0.3)
 		(layer "F.Cu")
@@
 	)
 	(segment
-		(start 36.3625 54.0125)
-		(end 36.3625 45.2625)
-		(width 0.3)
-		(layer "F.Cu")
-		(net 36)
-	)
-	(segment
-		(start 36.3625 45.2625)
-		(end 35.2625 44.1625)
+		(start 35.5125 48.4875)
+		(end 35.5125 54.7525)
 		(width 0.3)
 		(layer "F.Cu")
@@
 	)
 	(segment
-		(start 35.6225 54.7525)
-		(end 36.3625 54.0125)
+		(start 37.2625 43.1375)
+		(end 37.2625 46.7375)
 		(width 0.3)
 		(layer "F.Cu")
@@
 	)
 	(segment
-		(start 35.3625 45.7125)
-		(end 34.7625 45.1125)
-		(width 0.3)
-		(layer "F.Cu")
-		(net 37)
-	)
-	(segment
-		(start 34.5125 52.4625)
-		(end 35.3625 51.6125)
+		(start 34.5125 48.0875)
+		(end 34.5125 52.4625)
 		(width 0.3)
 		(layer "F.Cu")
@@
 	)
 	(segment
-		(start 35.3625 51.6125)
-		(end 35.3625 45.7125)
+		(start 36.7625 45.8375)
+		(end 34.5125 48.0875)
 		(width 0.3)
 		(layer "F.Cu")
@@
 	)
 	(segment
-		(start 34.7625 45.1125)
-		(end 34.7625 43.1375)
+		(start 36.7625 43.1375)
+		(end 36.7625 45.8375)
 		(width 0.3)
 		(layer "F.Cu")
@@
 	)
 	(segment
-		(start 33.5125 52.4625)
-		(end 33.5125 47.5125)
+		(start 35.2625 45.975)
+		(end 33.5125 47.725)
 		(width 0.3)
 		(layer "F.Cu")
@@
 	)
 	(segment
-		(start 34.2625 46.7625)
-		(end 34.2625 43.1375)
+		(start 33.5125 47.725)
+		(end 33.5125 52.4625)
 		(width 0.3)
 		(layer "F.Cu")
@@
 	)
 	(segment
-		(start 33.5125 47.5125)
-		(end 34.2625 46.7625)
+		(start 35.2625 43.1375)
+		(end 35.2625 45.975)
 		(width 0.3)
 		(layer "F.Cu")
@@
 	)
 	(segment
-		(start 32.5125 47.0375)
-		(end 33.7625 45.7875)
+		(start 32.5125 47.3875)
+		(end 32.5125 52.4625)
 		(width 0.3)
 		(layer "F.Cu")
@@
 	)
 	(segment
-		(start 33.7625 45.7875)
-		(end 33.7625 43.1375)
+		(start 34.7625 45.1375)
+		(end 32.5125 47.3875)
 		(width 0.3)
 		(layer "F.Cu")
@@
 	)
 	(segment
-		(start 32.5125 52.4625)
-		(end 32.5125 47.0375)
+		(start 34.7625 43.1375)
+		(end 34.7625 45.1375)
 		(width 0.3)
 		(layer "F.Cu")
