File: STM32_FlightController_Rev2/STM32_FlightController.kicad_sch (KiCad schematic)
At the start: 56 parts, among them J1 629105150521, J2 JST_SH_SM08B-SRSS-TB_1x08-1MP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, J3 JST_SH_SM04B-SRSS-TB_1x04-1MP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, J4 JST_SH_SM04B-SRSS-TB_1x04-1MP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, J5 Conn_02x05_Odd_Even, SW1 PTS815SJM250SMTRLFS, SW2 PCM12SMTR, U1 SN74LVC1T45DBV, U2 ICM-20948, U3 STM32F405RGTx, U4 USBLC6-2SC6, U5 AMS1117-3.3, U6 TLV70018, U7 BMP390L, U8 SN74LVC1T45DBV, Y1 X32258MOB4SI

Commit message: correct PCB traces regarding TIM pins
Connections:
- net S1: now also U3.27 (PB1); no longer U3.23 (PA7)
- net S2: now also U3.26 (PB0); no longer U3.22 (PA6)
- net S3: now also U3.23 (PA7); no longer U3.21 (PA5)
- net S4: now also U3.22 (PA6); no longer U3.20 (PA4)
Changed lines of the file:
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@@
 	)
 	(no_connect
+		(at 236.22 45.72)
+	)
+	(no_connect
+		(at 236.22 43.18)
+	)
+	(no_connect
 		(at 195.58 73.66)
 	)
@@
 	)
 	(no_connect
-		(at 236.22 78.74)
-	)
-	(no_connect
 		(at 236.22 35.56)
 	)
@@
 	)
 	(no_connect
-		(at 236.22 76.2)
-	)
-	(no_connect
 		(at 236.22 99.06)
 	)
@@
 	(wire
 		(pts
+			(xy 236.22 76.2) (xy 246.38 76.2)
+		)
+		(stroke
+			(width 0)
+			(type default)
+		)
+	)
+	(wire
+		(pts
 			(xy 195.58 99.06) (xy 176.53 99.06)
 		)
@@
 	(wire
 		(pts
+			(xy 236.22 78.74) (xy 246.38 78.74)
+		)
+		(stroke
+			(width 0)
+			(type default)
+		)
+	)
+	(wire
+		(pts
 			(xy 127 214.63) (xy 127 215.9)
 		)
@@
 	(wire
 		(pts
+			(xy 236.22 50.8) (xy 246.38 50.8)
+		)
+		(stroke
+			(width 0)
+			(type default)
+		)
+	)
+	(wire
+		(pts
 			(xy 35.56 78.74) (xy 36.83 78.74)
 		)
@@
 	(wire
 		(pts
+			(xy 236.22 48.26) (xy 246.38 48.26)
+		)
+		(stroke
+			(width 0)
+			(type default)
+		)
+	)
+	(wire
+		(pts
 			(xy 111.76 220.98) (xy 101.6 220.98)
 		)
@@
 	(wire
 		(pts
-			(xy 236.22 48.26) (xy 246.38 48.26)
-		)
-		(stroke
-			(width 0)
-			(type default)
-		)
-	)
-	(wire
-		(pts
 			(xy 236.22 88.9) (xy 246.38 88.9)
 		)
@@
 	(wire
 		(pts
-			(xy 236.22 50.8) (xy 246.38 50.8)
-		)
-		(stroke
-			(width 0)
-			(type default)
-		)
-	)
-	(wire
-		(pts
 			(xy 106.68 196.85) (xy 116.84 196.85)
 		)
@@
 	(wire
 		(pts
-			(xy 236.22 45.72) (xy 246.38 45.72)
-		)
-		(stroke
-			(width 0)
-			(type default)
-		)
-	)
-	(wire
-		(pts
 			(xy 19.05 204.47) (xy 19.05 205.74)
 		)
@@
 	(wire
 		(pts
-			(xy 236.22 43.18) (xy 246.38 43.18)
-		)
-		(stroke
-			(width 0)
-			(type default)
-		)
-	)
-	(wire
-		(pts
 			(xy 396.24 120.65) (xy 396.24 111.76)
 		)
@@
 		)
 	)
-	(label "S3"
-		(at 246.38 45.72 180)
-		(effects
-			(font
-				(size 1.27 1.27)
-			)
-			(justify right bottom)
-		)
-	)
 	(label "GPS_TX"
 		(at 246.38 40.64 180)
@@
 		)
 	)
-	(label "S4"
-		(at 246.38 43.18 180)
-		(effects
-			(font
-				(size 1.27 1.27)
-			)
-			(justify right bottom)
-		)
-	)
 	(label "INT2"
 		(at 185.42 76.2 0)
@@
 		)
 	)
+	(label "S4"
+		(at 246.38 48.26 180)
+		(effects
+			(font
+				(size 1.27 1.27)
+			)
+			(justify right bottom)
+		)
+	)
 	(label "IMU_MISO"
 		(at 355.6 52.07 0)
@@
 		)
 	)
-	(label "IMU_CS"
-		(at 355.6 59.69 0)
+	(label "S2"
+		(at 246.38 76.2 180)
 		(effects
 			(font
 				(size 1.27 1.27)
 			)
-			(justify left bottom)
+			(justify right bottom)
 		)
 	)
-	(label "INT1"
-		(at 185.42 78.74 0)
+	(label "IMU_CS"
+		(at 355.6 59.69 0)
 		(effects
 			(font
@@
 		)
 	)
-	(label "S1"
-		(at 246.38 50.8 180)
+	(label "INT1"
+		(at 185.42 78.74 0)
 		(effects
 			(font
 				(size 1.27 1.27)
 			)
-			(justify right bottom)
+			(justify left bottom)
 		)
 	)
@@
 		)
 	)
+	(label "S3"
+		(at 246.38 50.8 180)
+		(effects
+			(font
+				(size 1.27 1.27)
+			)
+			(justify right bottom)
+		)
+	)
 	(label "USB_D-"
 		(at 55.88 76.2 180)
@@
 		)
 	)
-	(label "S2"
-		(at 246.38 48.26 180)
+	(label "HSE_OUT"
+		(at 185.42 45.72 0)
 		(effects
 			(font
 				(size 1.27 1.27)
 			)
-			(justify right bottom)
+			(justify left bottom)
 		)
 	)
-	(label "HSE_OUT"
-		(at 185.42 45.72 0)
+	(label "S1"
+		(at 246.38 78.74 180)
 		(effects
 			(font
 				(size 1.27 1.27)
 			)
-			(justify left bottom)
+			(justify right bottom)
 		)
 	)
